File: LEVIA_H7.kicad_sch (KiCad schematic)
At the start: 9 parts, among them U1 USBLC6-2P6

Commit message: smaller OSD xtal
Parts:
- removed USB2: GT-USB-7095C, EasyEDA:USB-C-SMD_GT-USB-7095C, symbol EasyEDA:GT-USB-7095C
Connections:
- net GND: now also R2.2
- net USB_OTG.DM: now also U1.3 (I/O2), USB1.A7 (D-), USB1.B7 (D-); no longer U1.4 (I/O2)
- net USB_OTG.DP: now also U1.1 (I/O1), USB1.A6 (D+), USB1.B6 (D+); no longer U1.6 (I/O1)
- new net USB_OTG_P.DM: U1.4 (I/O2)
- new net USB_OTG_P.DP: U1.6 (I/O1)
Other:
- sheet MCU ports: added USB_OTG_P{USB}; removed USB_OTG{USB}
Changed lines of the file:
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@@
 	)
 	(junction
-		(at 68.58 58.42)
+		(at 67.31 58.42)
 		(diameter 0)
 		(color 0 0 0 0)
 	)
 	(junction
-		(at 68.58 55.88)
+		(at 67.31 55.88)
+		(diameter 0)
+		(color 0 0 0 0)
+	)
+	(junction
+		(at 80.01 48.26)
 		(diameter 0)
 		(color 0 0 0 0)
@@
 	(wire
 		(pts
-			(xy 66.04 55.88) (xy 68.58 55.88)
+			(xy 95.25 55.88) (xy 111.76 55.88)
+		)
+		(stroke
+			(width 0)
+			(type default)
+		)
+	)
+	(wire
+		(pts
+			(xy 95.25 58.42) (xy 111.76 58.42)
+		)
+		(stroke
+			(width 0)
+			(type default)
+		)
+	)
+	(wire
+		(pts
+			(xy 66.04 55.88) (xy 67.31 55.88)
 		)
 		(stroke
@@
 	(wire
 		(pts
-			(xy 80.01 45.72) (xy 80.01 49.53)
+			(xy 80.01 45.72) (xy 80.01 48.26)
 		)
 		(stroke
@@
 	(wire
 		(pts
-			(xy 68.58 58.42) (xy 85.09 58.42)
-		)
-		(stroke
-			(width 0)
-			(type default)
-		)
-	)
-	(wire
-		(pts
-			(xy 66.04 53.34) (xy 68.58 53.34)
+			(xy 67.31 58.42) (xy 85.09 58.42)
+		)
+		(stroke
+			(width 0)
+			(type default)
+		)
+	)
+	(wire
+		(pts
+			(xy 66.04 53.34) (xy 67.31 53.34)
 		)
 		(stroke
@@
 	(wire
 		(pts
-			(xy 68.58 60.96) (xy 68.58 58.42)
+			(xy 67.31 60.96) (xy 67.31 58.42)
 		)
 		(stroke
@@
 		)
 	)
-	(wire
-		(pts
-			(xy 95.25 55.88) (xy 111.76 55.88)
-		)
-		(stroke
-			(width 0)
-			(type default)
-		)
-	)
 	(bus
 		(pts
@@
 		)
 	)
-	(wire
-		(pts
-			(xy 95.25 58.42) (xy 111.76 58.42)
-		)
-		(stroke
-			(width 0)
-			(type default)
-		)
-	)
 	(bus
 		(pts
@@
 	(wire
 		(pts
-			(xy 66.04 60.96) (xy 68.58 60.96)
-		)
-		(stroke
-			(width 0)
-			(type default)
-		)
-	)
-	(wire
-		(pts
-			(xy 66.04 58.42) (xy 68.58 58.42)
+			(xy 66.04 60.96) (xy 67.31 60.96)
+		)
+		(stroke
+			(width 0)
+			(type default)
+		)
+	)
+	(wire
+		(pts
+			(xy 66.04 58.42) (xy 67.31 58.42)
 		)
 		(stroke
@@
 	(wire
 		(pts
-			(xy 68.58 55.88) (xy 85.09 55.88)
+			(xy 67.31 55.88) (xy 85.09 55.88)
 		)
 		(stroke
@@
 	(wire
 		(pts
-			(xy 68.58 53.34) (xy 68.58 55.88)
+			(xy 67.31 53.34) (xy 67.31 55.88)
 		)
 		(stroke
@@
 		)
 	)
-	(label "USB_OTG.DP"
-		(at 97.79 55.88 0)
+	(label "USB_OTG_P.DP"
+		(at 95.25 55.88 0)
 		(effects
 			(font
@@
 		)
 	)
+	(label "USB_OTG.DP"
+		(at 69.85 55.88 0)
+		(effects
+			(font
+				(size 1.27 1.27)
+			)
+			(justify left bottom)
+		)
+	)
 	(label "USB_OTG.DM"
-		(at 97.79 58.42 0)
+		(at 69.85 58.42 0)
+		(effects
+			(font
+				(size 1.27 1.27)
+			)
+			(justify left bottom)
+		)
+	)
+	(label "USB_OTG_P.DM"
+		(at 95.25 58.42 0)
 		(effects
 			(font
@@
 	(symbol
 		(lib_id "power:GND")
-		(at 80.01 49.53 0)
+		(at 80.01 48.26 0)
 		(unit 1)
 		(body_style 1)
@@
 		(dnp no)
 		(property "Reference" "#PWR02"
-			(at 80.01 55.88 0)
+			(at 80.01 54.61 0)
 			(hide yes)
 			(show_name no)
@@
 		)
 		(property "Value" "GND"
-			(at 78.74 53.34 0)
+			(at 78.74 52.07 0)
 			(show_name no)
 			(do_not_autoplace no)
@@
 		)
 		(property "Footprint" ""
-			(at 80.01 49.53 0)
+			(at 80.01 48.26 0)
 			(hide yes)
 			(show_name no)
@@
 		)
 		(property "Datasheet" ""
-			(at 80.01 49.53 0)
+			(at 80.01 48.26 0)
 			(hide yes)
 			(show_name no)
@@
 		)
 		(property "Description" "Power symbol creates a global label with name \"GND\" , ground"
-			(at 80.01 49.53 0)
+			(at 80.01 48.26 0)
 			(hide yes)
 			(show_name no)
@@
 	)
 	(symbol
-		(lib_id "EasyEDA:GT-USB-7095C")
-		(at 41.91 116.84 0)
-		(unit 1)
-		(body_style 1)
-		(exclude_from_sim no)
-		(in_bom yes)
-		(on_board yes)
-		(in_pos_files yes)
-		(dnp no)
-		(fields_autoplaced yes)
-		(property "Reference" "USB2"
-			(at 40.64 90.17 0)
-			(show_name no)
-			(do_not_autoplace no)
-			(effects
-				(font
-					(size 1.27 1.27)
-				)
-			)
-		)
-		(property "Value" "GT-USB-7095C"
-			(at 40.64 92.71 0)
-			(show_name no)
-			(do_not_autoplace no)
-			(effects
-				(font
-					(size 1.27 1.27)
-				)
-			)
-		)
-		(property "Footprint" "EasyEDA:USB-C-SMD_GT-USB-7095C"
-			(at 41.91 143.51 0)
-			(hide yes)
-			(show_name no)
-			(do_not_autoplace no)
-			(effects
-				(font
-					(size 1.27 1.27)
-				)
-			)
-		)
-		(property "Datasheet" "https://www.lcsc.com/datasheet/C22387147.pdf"
-			(at 41.91 146.05 0)
-			(hide yes)
-			(show_name no)
-			(do_not_autoplace no)
-			(effects
-				(font
-					(size 1.27 1.27)
-				)
-			)
-		)
-		(property "Description" ""
-			(at 41.91 116.84 0)
-			(hide yes)
-			(show_name no)
-			(do_not_autoplace no)
-			(effects
-				(font
-					(size 1.27 1.27)
-				)
-			)
-		)
-		(property "Manufacturer" "G-Switch(品赞)"
-			(at 41.91 148.59 0)
-			(hide yes)
-			(show_name no)
-			(do_not_autoplace no)
-			(effects
-				(font
-					(size 1.27 1.27)
-				)
-			)
-		)
-		(property "MPN" "GT-USB-7095C"
-			(at 41.91 151.13 0)
-			(hide yes)
-			(show_name no)
-			(do_not_autoplace no)
-			(effects
-				(font
-					(size 1.27 1.27)
-				)
-			)
-		)
-		(property "LCSC Part" "C22387147"
-			(at 41.91 153.67 0)
-			(hide yes)
-			(show_name no)
-			(do_not_autoplace no)
-			(effects
-				(font
-					(size 1.27 1.27)
-				)
-			)
-		)
-		(pin "A4"
-		)
-		(pin "A1"
-		)
-		(pin "A5"
-		)
-		(pin "A8"
-		)
-		(pin "A7"
-		)
-		(pin "A6"
-		)
-		(pin "2"
-		)
-		(pin "B6"
-		)
-		(pin "B9"
-		)
-		(pin "B7"
-		)
-		(pin "B8"
-		)
-		(pin "B12"
-		)
-		(pin "B1"
-		)
-		(pin "B5"
-		)
-		(pin "B4"
-		)
-		(pin "A12"
-		)
-		(pin "A9"
-		)
-		(instances
-			(project "LEVIA_H7"
-				(path "/6b768b36-fce6-4be0-9021-6d41bddc3a70"
-					(reference "USB2")
-					(unit 1)
-				)
-			)
-		)
-	)
-	(symbol
 		(lib_id "power:GND")
 		(at 114.3 176.53 0)
@@
 			)
 		)
-		(pin "USB_OTG{USB}" input
-			(at 120.65 53.34 180)
-			(effects
-				(font
-					(size 1.27 1.27)
-				)
-				(justify left)
-			)
-		)
 		(pin "ADC_AIRS" input
 			(at 120.65 82.55 180)
@@
 			(effects
 				(font
+					(size 1.27 1.27)
+				)
+				(justify left)
+			)
+		)
+		(pin "USB_OTG_P{USB}" input
+			(at 120.65 53.34 180)
+			(effects
+				(font

Commit message: layout attempts
Parts:
- H1, H2, H3, H4: now not fitted
Changed lines of the file:
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@@
 		(exclude_from_sim no)
 		(in_bom no)
-		(on_board yes)
-		(in_pos_files yes)
-		(dnp no)
+		(on_board no)
+		(in_pos_files no)
+		(dnp yes)
 		(fields_autoplaced yes)
 		(property "Reference" "H2"
@@
 		(exclude_from_sim no)
 		(in_bom no)
-		(on_board yes)
-		(in_pos_files yes)
-		(dnp no)
+		(on_board no)
+		(in_pos_files no)
+		(dnp yes)
 		(fields_autoplaced yes)
 		(property "Reference" "H1"
@@
 		(exclude_from_sim no)
 		(in_bom no)
-		(on_board yes)
-		(in_pos_files yes)
-		(dnp no)
+		(on_board no)
+		(in_pos_files no)
+		(dnp yes)
 		(fields_autoplaced yes)
 		(property "Reference" "H3"
@@
 		(exclude_from_sim no)
 		(in_bom no)
-		(on_board yes)
-		(in_pos_files yes)
-		(dnp no)
+		(on_board no)
+		(in_pos_files no)
+		(dnp yes)
 		(fields_autoplaced yes)
 		(property "Reference" "H4"
