File: ANALOG_VTX.kicad_sch (KiCad schematic)
At the start: 13 parts, among them U10 ZX-SH1.0-4PWT, U11 ZX-SH1.0-3PWT, U9 AT7456ELAH, Y2 XL2EL89COI-111YLC-27M

Commit message: smaller OSD xtal
Parts:
- Y2: value XL2EL89COI-111YLC-27M -> XL7EL89COI-111YLC-27M; footprint EasyEDA:CRYSTAL-SMD_4P-L3.2-W2.5-BL_SIT8008BI -> Crystal:Crystal_SMD_2016-4Pin_2.0x1.6mm; LCSC Part C5444553 -> C18214311; MPN XL2EL89COI-111YLC-27M -> XL7EL89COI-111YLC-27M
Changed lines of the file:
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@@
 			)
 		)
-		(property "Value" "XL2EL89COI-111YLC-27M"
+		(property "Value" "XL7EL89COI-111YLC-27M"
 			(at 93.98 74.93 0)
 			(hide yes)
@@
 			)
 		)
-		(property "Footprint" "EasyEDA:CRYSTAL-SMD_4P-L3.2-W2.5-BL_SIT8008BI"
+		(property "Footprint" "Crystal:Crystal_SMD_2016-4Pin_2.0x1.6mm"
 			(at 86.36 74.93 0)
 			(hide yes)
@@
 			)
 		)
-		(property "Datasheet" "https://www.lcsc.com/datasheet/C5444553.pdf"
+		(property "Datasheet" "https://www.lcsc.com/datasheet/C18214311.pdf"
 			(at 86.36 74.93 0)
 			(hide yes)
@@
 			)
 		)
-		(property "MPN" "XL2EL89COI-111YLC-27M"
+		(property "MPN" "XL7EL89COI-111YLC-27M"
 			(at 68.58 74.93 0)
 			(hide yes)
@@
 			)
 		)
-		(property "LCSC Part" "C5444553"
+		(property "LCSC Part" "C18214311"
 			(at 66.04 74.93 0)
 			(hide yes)

Commit message: BOM LCSC numbers assigned
Parts:
- C33, C34, C35, C38: LCSC Part (none) -> C1525
- C36, C37: LCSC Part (none) -> C15525
- R21: LCSC Part (none) -> C25744
- R22, R23: LCSC Part (none) -> C25133
Changed lines of the file:
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@@
+			)
+		)
+		(property "LCSC Part" "C25133"
+			(at 148.59 76.2 0)
+			(hide yes)
+			(show_name no)
+			(do_not_autoplace no)
+			(effects
+				(font
+					(size 1.27 1.27)
+				)
 			)
 		)
@@
 			)
 		)
+		(property "LCSC Part" "C1525"
+			(at 135.89 72.39 90)
+			(hide yes)
+			(show_name no)
+			(do_not_autoplace no)
+			(effects
+				(font
+					(size 1.27 1.27)
+				)
+			)
+		)
 		(pin "1"
 		)
@@
 			)
 		)
+		(property "LCSC Part" "C1525"
+			(at 63.5 48.26 0)
+			(hide yes)
+			(show_name no)
+			(do_not_autoplace no)
+			(effects
+				(font
+					(size 1.27 1.27)
+				)
+			)
+		)
 		(pin "1"
 		)
@@
 			)
 		)
+		(property "LCSC Part" "C15525"
+			(at 135.89 40.64 90)
+			(hide yes)
+			(show_name no)
+			(do_not_autoplace no)
+			(effects
+				(font
+					(size 1.27 1.27)
+				)
+			)
+		)
 		(pin "1"
 		)
@@
 		(property "Description" "Resistor, small symbol"
 			(at 148.59 36.83 0)
+			(hide yes)
+			(show_name no)
+			(do_not_autoplace no)
+			(effects
+				(font
+					(size 1.27 1.27)
+				)
+			)
+		)
+		(property "LCSC Part" "C25133"
+			(at 148.59 36.83 90)
 			(hide yes)
 			(show_name no)
@@
 			)
 		)
+		(property "LCSC Part" "C1525"
+			(at 53.34 39.37 0)
+			(hide yes)
+			(show_name no)
+			(do_not_autoplace no)
+			(effects
+				(font
+					(size 1.27 1.27)
+				)
+			)
+		)
 		(pin "1"
 		)
@@
 			)
 		)
+		(property "LCSC Part" "C1525"
+			(at 73.66 57.15 0)
+			(hide yes)
+			(show_name no)
+			(do_not_autoplace no)
+			(effects
+				(font
+					(size 1.27 1.27)
+				)
+			)
+		)
 		(pin "1"
 		)
@@
 		(property "Description" "Unpolarized capacitor, small symbol"
 			(at 135.89 36.83 0)
+			(hide yes)
+			(show_name no)
+			(do_not_autoplace no)
+			(effects
+				(font
+					(size 1.27 1.27)
+				)
+			)
+		)
+		(property "LCSC Part" "C15525"
+			(at 135.89 36.83 90)
 			(hide yes)
 			(show_name no)
@@
 			(hide yes)
 			(show_name no)
+			(do_not_autoplace no)
+			(effects
+				(font
+					(size 1.27 1.27)
+				)
+			)
+		)
+		(property "LCSC Part" "C25744"
+			(at 73.66 68.58 90)
+			(hide yes)
+			(show_name no)
