File: BUZZER.kicad_sch (KiCad schematic)
At the start: 4 parts, among them Q1 AO3400A, U21 ZX-SH1.0-3PWT

Commit message: BOM LCSC numbers assigned
Parts:
- Q1: LCSC Part (none) -> C20917
- R34: LCSC Part (none) -> C11702
- R35: LCSC Part (none) -> C25744
Changed lines of the file:
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@@
+			)
+		)
+		(property "LCSC Part" "C25744"
+			(at 93.98 66.04 0)
+			(hide yes)
+			(show_name no)
+			(do_not_autoplace no)
+			(effects
+				(font
+					(size 1.27 1.27)
+				)
 			)
 		)
@@
 			)
 		)
+		(property "LCSC Part" "C11702"
+			(at 88.9 62.23 90)
+			(hide yes)
+			(show_name no)
+			(do_not_autoplace no)
+			(effects
+				(font
+					(size 1.27 1.27)
+				)
+			)
+		)
 		(pin "2"
 		)
@@
 			(at 101.6 62.23 0)
 			(hide yes)
+			(show_name no)
+			(do_not_autoplace no)
+			(effects
+				(font
+					(size 1.27 1.27)
+				)
+			)
+		)
+		(property "LCSC Part" "C20917"
+			(at 101.6 62.23 0)
+			(hide yes)
