File: I2C1|SPI3.kicad_sch (KiCad schematic)
At the start: 6 parts, among them U18 ZX-SH1.0-4PWT, U19 ZX-SH1.0-6PWT

Commit message: BME280
Parts:
- R33: now not fitted; now left out of the parts list
Changed lines of the file:
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@@
 		(body_style 1)
 		(exclude_from_sim no)
-		(in_bom yes)
-		(on_board yes)
-		(in_pos_files yes)
-		(dnp no)
+		(in_bom no)
+		(on_board no)
+		(in_pos_files no)
+		(dnp yes)
 		(property "Reference" "R33"
 			(at 34.29 72.39 90)

Commit message: BOM LCSC numbers assigned
Parts:
- R30, R31: LCSC Part (none) -> C25900
- R32: LCSC Part (none) -> C25744
Changed lines of the file:
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@@
+			)
+		)
+		(property "LCSC Part" "C25900"
+			(at 38.1 67.31 90)
+			(hide yes)
+			(show_name no)
+			(do_not_autoplace no)
+			(effects
+				(font
+					(size 1.27 1.27)
+				)
 			)
 		)
@@
 			)
 		)
+		(property "LCSC Part" "C25900"
+			(at 38.1 64.77 90)
+			(hide yes)
+			(show_name no)
+			(do_not_autoplace no)
+			(effects
+				(font
+					(size 1.27 1.27)
+				)
+			)
+		)
 		(pin "2"
 		)
@@
 			(hide yes)
 			(show_name no)
+			(do_not_autoplace no)
+			(effects
+				(font
+					(size 1.27 1.27)
+				)
+			)
+		)
+		(property "LCSC Part" "C25744"
+			(at 38.1 71.12 90)
+			(hide yes)
+			(show_name no)
